Commit message: Gazebo additions

File: description/robot.urdf.xacro (robot description, xacro)
@@ -2,3 +2,4 @@
 <robot xmlns:xacro="http://www.ros.org/wiki/xacro"  name="robot">
     <xacro:include filename="/home/fe25/dev_ws/src/my_bot/description/robot_core.xacro"/>
+    <xacro:include filename="/home/fe25/dev_ws/src/my_bot/description/gazebo_control.xacro"/>
 </robot>

File: description/robot_core.xacro (robot description, xacro)
@@ -41,4 +41,7 @@
         </xacro:inertial_box>
     </link>
+    <gazebo reference="chassis">
+        <material>Gazebo/White</material>
+    </gazebo>
     <!-- BACK LEFT WHEEL LINK-->
     <joint name="back_left_wheel_joint" type="continuous">
@@ -64,4 +67,7 @@
         </xacro:inertial_cylinder>
     </link>
+    <gazebo reference="back_left_wheel">
+        <material>Gazebo/Blue</material>
+    </gazebo>
     <!-- BACK RIGHT WHEEL LINK-->
     <joint name="back_right_wheel_joint" type="continuous">
@@ -87,4 +93,7 @@
         </xacro:inertial_cylinder>
     </link>
+    <gazebo reference="back_right_wheel">
+        <material>Gazebo/Blue</material>
+    </gazebo>
     <!-- FRONT LEFT WHEEL LINK -->
     <joint name="front_left_wheel_joint" type="revolute">
@@ -111,4 +120,9 @@
         </xacro:inertial_cylinder>
     </link>
+    <gazebo reference="front_left_wheel">
+        <material>Gazebo/Blue</material>
+        <mu1 value="0.0001"/>
+        <mu2 value="0.0001"/>
+    </gazebo>
     <!-- FRONT RIGHT WHEEL LINK -->
     <joint name="front_right_wheel_joint" type="revolute">
@@ -135,3 +149,8 @@
         </xacro:inertial_cylinder>
     </link>
+    <gazebo reference="front_right_wheel">
+        <material>Gazebo/Blue</material>
+        <mu1 value="0.0001"/>
+        <mu2 value="0.0001"/>
+    </gazebo>
 </robot>

Commit message: Add ros2_control and dynamixel_hardware initialisation

File: description/robot.urdf.xacro (robot description, xacro)
@@ -1,6 +1,7 @@
 <?xml version="1.0"?>
 <robot xmlns:xacro="http://www.ros.org/wiki/xacro"  name="robot">
-    <xacro:include filename="/home/fe25/dev_ws/src/my_bot/description/robot_core.xacro"/>
-    <xacro:include filename="/home/fe25/dev_ws/src/my_bot/description/gazebo_control.xacro"/>
-    <xacro:include filename="/home/fe25/dev_ws/src/my_bot/description/lidar.xacro"/>
+    <xacro:include filename="ros2_control.xacro"/>
+    <!--<xacro:include filename="gazebo_control.xacro"/>-->
+    <xacro:include filename="robot_core.xacro"/>
+    <xacro:include filename="lidar.xacro"/>
 </robot>

File: description/robot_core.xacro (robot description, xacro)
@@ -27,5 +27,5 @@
             <origin xyz="0.05 0 0.05"></origin>
             <geometry>
-                <box size="0.3 0.15 0.15" />
+                <box size="0.3 0.15 0.10" />
             </geometry>
             <material name="white"/>
@@ -34,8 +34,8 @@
             <origin xyz="0.05 0 0.05"></origin>
             <geometry>
-                <box size="0.3 0.15 0.15" />
+                <box size="0.3 0.15 0.10" />
             </geometry>
         </collision>
-        <xacro:inertial_box mass="0.85" x="0.3" y="0.15" z="0.15">
+        <xacro:inertial_box mass="0.85" x="0.3" y="0.15" z="0.10">
             <origin xyz="0.05 0 0.075"/>
         </xacro:inertial_box>
