Commit message: Remove gazebo

File: description/lidar.xacro (robot description, xacro)
@@ -29,26 +29,3 @@
         </xacro:inertial_cylinder>
     </link>
-    <gazebo reference="lidar_frame">
-        <material>Gazebo/Black</material>
-        <sensor name="lidar" type="gpu_lidar">
-            <pose> 0 0 0 0 0 0 </pose>
-            <visualize>false</visualize>
-            <update_rate>10</update_rate>
-            <lidar>
-                <scan>
-                    <horizontal>
-                        <samples>360</samples>
-                        <min_angle>-3.14</min_angle>
-                        <max_angle>3.14</max_angle>
-                    </horizontal>
-                </scan>
-                <range>
-                    <min>0.3</min>
-                    <max>12</max>
-                </range>
-            </lidar>
-            <topic>scan</topic>
-            <gz_frame_id>lidar_frame</gz_frame_id>
-        </sensor>
-    </gazebo>
 </robot>

File: description/robot.urdf.xacro (robot description, xacro)
@@ -2,5 +2,4 @@
 <robot xmlns:xacro="http://www.ros.org/wiki/xacro"  name="robot">
     <xacro:include filename="ros2_control.xacro"/>
-    <xacro:include filename="gazebo_control.xacro"/>
     <xacro:include filename="robot_core.xacro"/>
     <xacro:include filename="lidar.xacro"/>

File: description/robot_core.xacro (robot description, xacro)
@@ -41,7 +41,4 @@
         </xacro:inertial_box>
     </link>
-    <gazebo reference="chassis">
-        <material>Gazebo/White</material>
-    </gazebo>
     <!-- BACK LEFT WHEEL LINK-->
     <joint name="back_left_wheel_joint" type="continuous">
@@ -67,7 +64,4 @@
         </xacro:inertial_cylinder>
     </link>
-    <gazebo reference="back_left_wheel">
-        <material>Gazebo/Blue</material>
-    </gazebo>
     <!-- BACK RIGHT WHEEL LINK-->
     <joint name="back_right_wheel_joint" type="continuous">
@@ -93,7 +87,4 @@
         </xacro:inertial_cylinder>
     </link>
-    <gazebo reference="back_right_wheel">
-        <material>Gazebo/Blue</material>
-    </gazebo>
     <!-- FRONT LEFT WHEEL LINK -->
     <joint name="front_left_wheel_joint" type="revolute">
@@ -120,9 +111,4 @@
         </xacro:inertial_cylinder>
     </link>
-    <gazebo reference="front_left_wheel">
-        <material>Gazebo/Blue</material>
-        <mu1 value="0.0001"/>
-        <mu2 value="0.0001"/>
-    </gazebo>
     <!-- FRONT RIGHT WHEEL LINK -->
     <joint name="front_right_wheel_joint" type="revolute">
@@ -149,8 +135,3 @@
         </xacro:inertial_cylinder>
     </link>
-    <gazebo reference="front_right_wheel">
-        <material>Gazebo/Blue</material>
-        <mu1 value="0.0001"/>
-        <mu2 value="0.0001"/>
-    </gazebo>
 </robot>

File: description/ros2_control.xacro (robot description, xacro)
@@ -1,6 +1,5 @@
 <?xml version="1.0"?>
 <robot xmlns:xacro="http://www.ros.org/wiki/xacro">
-    <!--<ros2_control name="ros2_control" type="system"></ros2_control>-->
-    <ros2_control name="GazeboSystem" type="system">
+    <ros2_control name="ros2_control" type="system">
         <hardware>
             <plugin>gazebo_ros2_control/GazeboSystem</plugin>
@@ -38,8 +37,3 @@
         </joint>
     </ros2_control>
-    <gazebo>
-        <plugin name="gazebo_ros2_control" filename="libgazebo_ros2_control.so">
-            <parameters>$(find my_bot)/config/my_controllers.yaml</parameters>
-        </plugin>
-    </gazebo>
 </robot>
